Commit message: feat(stage-1): sanitize URDF meshes and implement MuJoCo MJCF model with sensors

File: urdf_model/root/urdf/root.urdf (robot description, URDF)
Before this commit: robot root, 8 links, 7 joints
Links:
- removed link base__spinningpart
- removed link base__подставка
- removed link elbow__main
- removed link robohandforsimback_x_t__Тело_110
- removed link shoulder__Импортировано_01__1_
- added link base_link, mass 0.140; collision mesh filename=../meshes/base_stand.stl scale=1 1 1; visual mesh filename=../meshes/base_stand.stl scale=1 1 1
- added link base_spinning, mass 0.135; collision mesh filename=../meshes/base_spinning.stl scale=1 1 1; visual mesh filename=../meshes/base_spinning.stl scale=1 1 1
- added link elbow_link, mass 0.110; collision mesh filename=../meshes/elbow.stl scale=1 1 1; visual mesh filename=../meshes/elbow.stl scale=1 1 1
- added link shoulder_link, mass 0.132; collision mesh filename=../meshes/shoulder.stl scale=1 1 1; visual mesh filename=../meshes/shoulder.stl scale=1 1 1
- added link wrist_link, mass 0.065; collision mesh filename=../meshes/wrist.stl scale=1 1 1; visual mesh filename=../meshes/wrist.stl scale=1 1 1
- link main__gripper1: mass 1.06918e-05 -> 0.015; geometry collision mesh filename=../meshes/gripper_finger1.stl scale=1 1 1; visual mesh filename=../meshes/gripper_finger1.stl scale=1 1 1
- link main__gripper2: mass 1.15881e-05 -> 0.015; geometry collision mesh filename=../meshes/gripper_finger2.stl scale=1 1 1; visual mesh filename=../meshes/gripper_finger2.stl scale=1 1 1
- link main__gripperbase: mass 8.61997e-06 -> 0.086; geometry collision mesh filename=../meshes/gripper_base.stl scale=1 1 1; visual mesh filename=../meshes/gripper_base.stl scale=1 1 1
Joints:
- joint revolute_1: child base__spinningpart -> base_spinning; limit (none) -> lower=-3.14159 upper=3.14159 effort=1.5 velocity=3.0; origin xyz=0 0 0.013 rpy=0 -0 0 -> xyz=0 0 0.013 rpy=0 0 0; parent base__подставка -> base_link; type continuous -> revolute
- joint revolute_2: child shoulder__Импортировано_01__1_ -> shoulder_link; limit lower=-1.5708 upper=1.5708 effort=1.0 velocity=3.0 -> lower=-1.5708 upper=1.5708 effort=2.5 velocity=3.0; origin xyz=-0.00153435 0.010669 0.043598 rpy=0 -0 0 -> xyz=-0.00153435 0.010669 0.043598 rpy=0 0 0; parent base__spinningpart -> base_spinning
- joint revolute_3: child elbow__main -> elbow_link; limit lower=-1.5708 upper=1.5708 effort=1.0 velocity=3.0 -> lower=-1.5708 upper=1.5708 effort=2.0 velocity=3.0; origin xyz=0 -1.94116e-15 0.117 rpy=0 -0 0 -> xyz=0 0 0.117 rpy=0 0 0; parent shoulder__Импортировано_01__1_ -> shoulder_link
- joint revolute_4: child robohandforsimback_x_t__Тело_110 -> wrist_link; limit lower=-1.5708 upper=1.5708 effort=1.0 velocity=3.0 -> lower=-1.5708 upper=1.5708 effort=1.5 velocity=3.0; origin xyz=-7.67294e-05 -0.0207719 0.117514 rpy=0 -0 0 -> xyz=-7.67294e-05 -0.0207719 0.117514 rpy=0 0 0; parent elbow__main -> elbow_link
- joint revolute_5: origin xyz=-0.0127233 0.0100928 0.0740668 rpy=0 -0 0 -> xyz=-0.0127233 0.0100928 0.0740668 rpy=0 0 0; parent robohandforsimback_x_t__Тело_110 -> wrist_link
- joint revolute_6: axis -0.999982 0.00605305 4.33681e-19 -> -1 0 0; origin xyz=-0.0042323 -0.00744957 0.0355 rpy=-7.16466e-17 -1.20371e-34 4.31208e-51 -> xyz=-0.0042323 -0.00744957 0.0355 rpy=0 0 0
- joint revolute_7: axis -0.999982 0.00605305 1.0842e-19 -> -1 0 0; origin xyz=-0.0041294 0.00955012 0.0355 rpy=-1.79117e-17 -3.61112e-35 3.23406e-52 -> xyz=-0.0041294 0.00955012 0.0355 rpy=0 0 0
