Commit message: refactor: consolidate all models and meshes into assets/ and remove urdf_model/

File: assets/root.urdf (robot description, URDF)
Before this commit: robot root, 8 links, 7 joints
Links:
- link base_link: geometry collision mesh filename=meshes/base_stand.stl scale=1 1 1; visual mesh filename=meshes/base_stand.stl scale=1 1 1
- link base_spinning: geometry collision mesh filename=meshes/base_spinning.stl scale=1 1 1; visual mesh filename=meshes/base_spinning.stl scale=1 1 1
- link elbow_link: geometry collision mesh filename=meshes/elbow.stl scale=1 1 1; visual mesh filename=meshes/elbow.stl scale=1 1 1
- link main__gripper1: geometry collision mesh filename=meshes/gripper_finger1.stl scale=1 1 1; visual mesh filename=meshes/gripper_finger1.stl scale=1 1 1
- link main__gripper2: geometry collision mesh filename=meshes/gripper_finger2.stl scale=1 1 1; visual mesh filename=meshes/gripper_finger2.stl scale=1 1 1
- link main__gripperbase: geometry collision mesh filename=meshes/gripper_base.stl scale=1 1 1; visual mesh filename=meshes/gripper_base.stl scale=1 1 1
- link shoulder_link: geometry collision mesh filename=meshes/shoulder.stl scale=1 1 1; visual mesh filename=meshes/shoulder.stl scale=1 1 1
- link wrist_link: geometry collision mesh filename=meshes/wrist.stl scale=1 1 1; visual mesh filename=meshes/wrist.stl scale=1 1 1

Commit message: feat(manipulator): implement Stage 7 ToF-assisted grasping and pick-and-place state machine

File: assets/root.urdf (robot description, URDF)
Before this commit: robot root, 8 links, 7 joints
Joints:
- joint revolute_6: limit lower=-0.6 upper=0.15 effort=1.0 velocity=3.0 -> lower=-0.6 upper=0.6 effort=1.0 velocity=3.0
- joint revolute_7: limit lower=-0.15 upper=0.6 effort=1.0 velocity=3.0 -> lower=-0.6 upper=0.6 effort=1.0 velocity=3.0
